File: hardware/myriad_0.2/myriad_0.2.kicad_sch (KiCad schematic)
At the start: 108 parts, among them J1 CV In 1, J10 ELI2040B 1, J2 CV In 2, J3 ELI2040B 1, J4 CV In 3, J5 CV In 4, J6 Clean Out, J7 Shaped Out, J8 Conn_01x02_Socket, J9 Conn_01x02_Socket, Q1 MMBT3906, Q2 MMBT3904, Q3 MMBT3906, Q4 MMBT3904, SW1 TS-1187A-B-A-B, U1 TL072, U2 MCP6002-xMS, U3 CJ431 SOT-23, U4 CJ431 SOT-23, U5 TL072, U6 TL072, U7 MCP6002-xMS, U8 TL072

Commit message: finally approaching multiple pitch control
Parts:
- added C21, C22: 100n, Capacitor_SMD:C_0603_1608Metric, symbol Device:C
- added R13, R14, R8: 33k, Resistor_SMD:R_0603_1608Metric, symbol Device:R
- added R24, R30, R35: 10k, Resistor_SMD:R_0603_1608Metric, symbol Device:R
- added R31: 5.1k, Resistor_SMD:R_0603_1608Metric, symbol Device:R
- added R36: 39k, Resistor_SMD:R_0603_1608Metric, symbol Device:R
- added U4: TL072, Package_SO:SO-8_3.9x4.9mm_P1.27mm, symbol Amplifier_Operational:TL072
- J1: renamed from J3; symbol emutelab:ELI2040_B -> emutelab:ELI2040_C
- J2: renamed from J10; symbol emutelab:ELI2040_B -> emutelab:ELI2040_C
- R11: renamed from R20; value 1.3k -> 1.2k
- R12: renamed from R23; value 1.3k -> 1.2k
- R33: renamed from R41; value 560 -> 2k
- renumbered C9 to C1, C17 to C10, C18 to C11, C19 to C12, C20 to C13, C21 to C14, C13 to C15, C7 to C16, C8 to C17, C25 to C18, C23 to C19, C12 to C2, C24 to C20, C5 to C3, C10 to C4, C11 to C5, C22 to C6, C14 to C7, C15 to C8, C16 to C9, D3 to D1, D4 to D2, J5 to J10, J6 to J3, J8 to J4, J9 to J5, J7 to J6, J4 to J7, J1 to J8, J2 to J9, R17 to R1, R48 to R10, R27 to R15, R29 to R16, R31 to R17, R9 to R18, R12 to R19, R18 to R2, R13 to R20, R14 to R21, R15 to R22, R16 to R23, R44 to R25, R33 to R26, R34 to R27, R36 to R28, R37 to R29, R19 to R3, R39 to R32, R45 to R34, R21 to R37, R1 to R38, R2 to R39, R22 to R4, R35 to R40, R26 to R41, R3 to R42, R4 to R43, R38 to R44, R28 to R45, R30 to R46, R5 to R47, R6 to R48, R40 to R49, R46 to R5, R7 to R50, R8 to R51, R42 to R52, R32 to R53, R10 to R54, R11 to R55, R43 to R56, R24 to R6, R25 to R7, R47 to R9, RV3 to RV1, RV1 to RV2, RV2 to RV3, RV5 to RV4, RV4 to RV4_Waveshape1, RV6 to RV6_Overdrive1, S2 to S1, S3 to S2, S1 to S3, TP2 to TP1, TP3 to TP2, TP1 to TP3, U9 to U1, U6 to U10, U3 to U2, U4 to U3, U8 to U6, U2 to U7, U7 to U8, U1 to U9
Connections:
- net +12V: now also C22.2, U4.4 (V-)
- net -12V: now also J2.1 (-12V), C21.2, U4.8 (V+)
- net GND: now also C21.1, C22.1, R31.2, R35.1, U4.5 (+); no longer J1.4 (Pin_4), J2.4 (Pin_4), RV4_Waveshape1.3
- net at R10.2, R11.1, R18.2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: now also R13.2, R14.2, R8.2
- net at R17.2, U5.7, U6.3 (+): now also R24.1; no longer RV4_Waveshape1.1
- net at J2.18 (Pin_18): now also R13.1
- net at J2.19 (Pin_19): now also R14.1
- net at J2.22 (Pin_22): now also J1.23 (Pin_23); no longer J1.22 (Pin_22)
- net at J2.23 (Pin_23): now also J1.22 (Pin_22); no longer J1.24 (Pin_24)
- net at J2.24 (Pin_24): no longer J1.23 (Pin_23)
- net at J2.25 (Pin_25): no longer J1.25 (Pin_25)
- net at Q1.1 (B), Q2.1 (B), RV4_Waveshape1.2: now also RV4_Waveshape1.3
- net at R5.1: now also J1.25 (Pin_25); no longer J1.28 (Pin_28)
- net at U6.5 (+): now also R30.2, R31.1; no longer J4.1 (Pin_1)
- net at C6.1, D1.2 (A), D2.1 (K)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: now also RV6_Overdrive1.1, U4.3 (+); no longer R34.1, RV6_Overdrive1.3
- net at R33.2: now also RV6_Overdrive1.3; no longer RV6_Overdrive1.1
- new net: U4.6 (-), U4.7
- new net: R24.2, RV4_Waveshape1.1
- new net: R35.2, R36.1, U4.2 (-)
- new net: R34.1, R36.2, U4.1
- new net: J4.1 (Pin_1), R30.1
- new net: J1.28 (Pin_28), R8.1
- no-connect marks 28 -> 27
Other:
- note added: "circuit JS link"
- moved on the sheet: C19, C20, J5, J6, R34, R5, RV6_Overdrive1, U6C
