File: hardware/panel/myriadPCBPanel_0.3/myriadPCBPanel_0.3.kicad_pcb (KiCad board)
At the start: 2 copper layers, 81.7 x 128.9 mm, 21 parts

Commit message: modulation targets
Parts:
- added REF**: PanelHole_AudioJack_3.5mm, benjiaomodular:PanelHole_AudioJack_3.5mm, F.Cu at (98.0, 122.8)
- moved REF** 70.6 mm to (87.7, 122.8)
- moved REF** 68.6 mm to (77.3, 122.8)
- moved REF** 66.4 mm to (67.0, 122.8)
- moved REF** 65.5 mm to (85.2, 50.4)
- moved REF** 64.6 mm to (95.2, 118.2)
- moved REF** 64.4 mm to (118.6, 122.8)
- moved REF** 64.4 mm to (56.7, 122.8)
- moved REF** 64.4 mm to (52.0, 149.5)
- moved REF** 64.4 mm to (121.2, 149.5)
- moved REF** 64.3 mm to (114.0, 51.4)
- moved REF** 64.3 mm to (56.1, 51.3)
- moved REF** 64.3 mm to (80.3, 70.8)
- moved REF** 64.3 mm to (52.0, 27.0)
- moved REF** 64.3 mm to (121.2, 27.0)
- moved REF** 64.3 mm to (57.1, 98.8)
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Other:
- board text added: "Myriad 0.3"
- board text removed: "Myriad 0.2"
