File: hardware/myriad_0.4/myriad_0.4.kicad_sch (KiCad schematic)
At the start: 114 parts, among them J1 CV Shape, J2 ELI2040B 1, J3 ELI2040B 1, J4 CV In 3, J5 CV In 1, J6 CV In 2, J7 CV In 4, Q1 MMBT3906, SW1 TS-1187A-B-A-B, SW2 SW_DPDT_x2, U10 TL074, U11 TL074, U12 TL074, U2 CJ431 SOT-23, U3 CJ431 SOT-23, U4 TL074, U5 LM13700, U6 TL072, U7 MCP6002-xMS, U8 TL074, U9 MCP6002-xMS

Commit message: separate LR outs
Parts:
- removed C6, C7: 100n, Capacitor_SMD:C_0603_1608Metric, symbol Device:C
- removed SW2: SW_DPDT_x2, symbol Switch:SW_DPDT_x2
- removed U6: TL072, Package_SO:SO-8_3.9x4.9mm_P1.27mm, symbol Amplifier_Operational:TL072
- added C36, C37: 100n, Capacitor_SMD:C_0603_1608Metric, symbol Device:C
- added J_Out_L2: Shape out L, Connector_Audio:Jack_3.5mm_QingPu_WQP-PJ398SM_Vertical_CircularHoles, symbol Connector:AudioJack2_SwitchT
- added J_Out_R2: Shape Out R, Connector_Audio:Jack_3.5mm_QingPu_WQP-PJ398SM_Vertical_CircularHoles, symbol Connector:AudioJack2_SwitchT
- added R86, R89: 68k, Resistor_SMD:R_0603_1608Metric, symbol Device:R
- added R87, R92: 47k, Resistor_SMD:R_0603_1608Metric, symbol Device:R
- added R88, R95: 1k, Resistor_SMD:R_0603_1608Metric, symbol Device:R
- added R90, R91: 10k, symbol Device:R
- added R93, R94: 100k, symbol Device:R
- added R96: 1k, symbol Device:R
- added U13: TL074, symbol Amplifier_Operational:TL074
- R9: value 51k -> 100k
Connections:
- net +12V: now also C37.2, U13.4 (V+)
- net -12V: now also C36.2, U13.11 (V-)
- net GND: now also C36.1, C37.1, J_Out_L2.S, J_Out_R2.S, R87.1, R92.1, R93.2, R94.2
- net Clean Out R: now reaches U8.3 (+)
- net Clean Out L: now reaches U8.5 (+)
- net at R33.1, U8.8: now also U8.9 (-)
- new net: J_Out_R2.T, R95.2
- new net: J_Out_R2.TN, R90.1
- new net: J_Out_L2.T, R96.2
- new net: R89.2, R92.2, R95.1, U13.1
- new net: R89.1, U13.2 (-)
- new net: R90.2, R91.2, R93.1, R94.1, U13.10 (+)
- new net: R96.1, U13.8, U13.9 (-)
- new net: R86.1, U13.6 (-)
- new net: R86.2, R87.2, R88.1, U13.7
- new net: R88.2, R91.1
- new net Shape Out L: U13.5 (+)
- new net Shape Out R: U13.3 (+)
- no-connect marks 30 -> 36
Other:
- sheet filter-vca ports: added +5V; removed none
- sheet filter-vca1 ports: added +5V; removed none
- note added: "0-1mA"
- note added: "10uA"
- note added: "500uA"
- note added: "R9/R14 is current gain, split across two OTAs"
- note removed: "clean gain/buffered out"
- note removed: "shaped gain/buffered out"
- moved on the sheet: J_Out_L1, J_Out_R1, R23, R24, R25, R26, R27, R28, R29, R30, R31, R32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

Commit message: almost routed
Parts:
- added unit 4 of U10
- added unit 4 of U13
- added unit 4 of U8
- R25, R26, R28, R29, R33, R90, R91, R93, R94, R96: footprint (none) -> Resistor_SMD:R_0603_1608Metric
- U10, U11, U12, U13, U4, U8: footprint (none) -> Package_SO:TSSOP-14_4.4x5mm_P0.65mm
- renumbered RV2-CV1 to RV-CV1, RV3-CV1 to RV-CV2, RV1-CV1 to RV-CV3, RV4-CV1 to RV-CV4
Connections:
- net GND: now also U10.12 (+), U13.12 (+), U8.12 (+)
- new net: U8.13 (-), U8.14
- new net: U10.13 (-), U10.14
- new net: U13.13 (-), U13.14

Commit message: v0.4 proto
Parts:
- R28, R29, R93, R94: value 100k -> 100k 0603
- R50, R51, R52, R53: value 33k -> 33k_0402
Changed lines of the file:
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@@
 		(fields_autoplaced yes)
 		(property "Reference" "R29"
-			(at 537.464 179.0701 0)
+			(at 533.4 176.5299 0)
 			(effects
 				(font
 					(size 1.27 1.27)
 				)
-				(justify left)
+				(justify right)
 			)
 		)
-		(property "Value" "100k"
-			(at 537.464 176.5301 0)
+		(property "Value" "100k 0603"
+			(at 533.4 179.0699 0)
 			(effects
 				(font
 					(size 1.27 1.27)
 				)
-				(justify left)
+				(justify right)
 			)
 		)
@@
 		(fields_autoplaced yes)
 		(property "Reference" "R51"
-			(at 771.525 91.8677 90)
+			(at 771.525 91.44 90)
 			(effects
 				(font
@@
 			)
 		)
-		(property "Value" "33k"
-			(at 771.525 94.2919 90)
+		(property "Value" "33k_0402"
+			(at 771.525 93.98 90)
 			(effects
 				(font
@@
 		(fields_autoplaced yes)
 		(property "Reference" "R50"
-			(at 770.255 206.1677 90)
+			(at 770.255 205.74 90)
 			(effects
 				(font
@@
 			)
 		)
-		(property "Value" "33k"
-			(at 770.255 208.5919 90)
+		(property "Value" "33k_0402"
+			(at 770.255 208.28 90)
 			(effects
 				(font
@@
 		(fields_autoplaced yes)
 		(property "Reference" "R94"
-			(at 540.258 321.6911 0)
+			(at 535.94 319.1509 0)
 			(effects
 				(font
 					(size 1.27 1.27)
 				)
-				(justify left)
+				(justify right)
 			)
 		)
-		(property "Value" "100k"
-			(at 540.258 319.1511 0)
+		(property "Value" "100k 0603"
+			(at 535.94 321.6909 0)
 			(effects
 				(font
 					(size 1.27 1.27)
 				)
-				(justify left)
+				(justify right)
 			)
 		)
@@
 		(fields_autoplaced yes)
 		(property "Reference" "R53"
-			(at 771.525 263.3177 90)
+			(at 771.525 262.89 90)
 			(effects
 				(font
@@
 			)
 		)
-		(property "Value" "33k"
-			(at 771.525 265.7419 90)
+		(property "Value" "33k_0402"
+			(at 771.525 265.43 90)
 			(effects
 				(font
@@
 		(fields_autoplaced yes)
 		(property "Reference" "R93"
-			(at 539.369 337.1849 0)
+			(at 539.75 337.1849 0)
 			(effects
 				(font
@@
 			)
 		)
-		(property "Value" "100k"
-			(at 539.369 339.7249 0)
+		(property "Value" "100k 0603"
+			(at 539.75 339.7249 0)
 			(effects
 				(font
@@
 		(fields_autoplaced yes)
 		(property "Reference" "R52"
-			(at 771.525 142.6677 90)
+			(at 771.525 142.24 90)
 			(effects
 				(font
@@
 			)
 		)
-		(property "Value" "33k"
-			(at 771.525 145.0919 90)
+		(property "Value" "33k_0402"
+			(at 771.525 144.78 90)
 			(effects
 				(font
@@
 		(fields_autoplaced yes)
 		(property "Reference" "R28"
-			(at 536.575 194.5639 0)
+			(at 537.21 194.5639 0)
 			(effects
 				(font
@@
 			)
 		)
-		(property "Value" "100k"
-			(at 536.575 197.1039 0)
+		(property "Value" "100k 0603"
+			(at 537.21 197.1039 0)
 			(effects
 				(font
